Commit message: modifique el multirotor_base.xacro para que admita lenght tambien y actualice todos los archivos que rompi con ese cambio

File: rotors_description/urdf/ardrone.xacro (robot description, xacro)
@@ -37,4 +37,6 @@
     robot_namespace="${namespace}"
     mass="${mass}"
+    use_body_length="false"
+    body_length=""
     body_width="${body_width}"
     body_height="${body_height}"

File: rotors_description/urdf/asymmetric_quadrotor.xacro (robot description, xacro)
@@ -50,4 +50,6 @@
     robot_namespace="${namespace}"
     mass="${mass}"
+    use_body_length="false"
+    body_length=""
     body_width="${body_width}"
     body_height="${body_height}"

File: rotors_description/urdf/firefly.xacro (robot description, xacro)
@@ -52,4 +52,6 @@
     robot_namespace="${namespace}"
     mass="${mass}"
+    use_body_length="false"
+    body_length=""
     body_width="${body_width}"
     body_height="${body_height}"

File: rotors_description/urdf/hummingbird.xacro (robot description, xacro)
@@ -51,4 +51,6 @@
     robot_namespace="${namespace}"
     mass="${mass}"
+    use_body_length="false"
+    body_length=""
     body_width="${body_width}"
     body_height="${body_height}"

File: rotors_description/urdf/iris.xacro (robot description, xacro)
@@ -40,4 +40,6 @@
     robot_namespace="${namespace}"
     mass="${mass}"
+    use_body_length="false"
+    body_length=""
     body_width="${body_width}"
     body_height="${body_height}"

File: rotors_description/urdf/multirotor_base.xacro (robot description, xacro)
@@ -33,5 +33,5 @@
   <!-- Main multirotor link -->
   <xacro:macro name="multirotor_base_macro"
-    params="robot_namespace mass body_width body_height use_mesh_file mesh_file *inertia">
+    params="robot_namespace mass body_width body_height use_body_length body_length use_mesh_file mesh_file *inertia">
     <link name="${robot_namespace}/base_link"></link>
     <joint name="${robot_namespace}/base_joint" type="fixed">
@@ -53,5 +53,10 @@
           </xacro:if>
           <xacro:unless value="${use_mesh_file}">
-            <box size="${body_width} ${body_width} ${body_height}"/> <!-- [m] [m] [m] -->
+            <xacro:if value="${use_body_length}">
+              <box size="${body_length} ${body_width} ${body_height}"/> <!-- [m] [m] [m] -->
+            </xacro:if>
+            <xacro:unless value="${use_body_length}">
+              <box size="${body_width} ${body_width} ${body_height}"/> <!-- [m] [m] [m] -->
+            </xacro:unless>
           </xacro:unless>
         </geometry>
@@ -60,5 +65,10 @@
         <origin xyz="0 0 0" rpy="0 0 0" />
         <geometry>
-          <box size="${body_width} ${body_width} ${body_height}" /> <!-- [m] [m] [m] -->
+          <xacro:if value="${use_body_length}">
+            <box size="${body_length} ${body_width} ${body_height}"/> <!-- [m] [m] [m] -->
+          </xacro:if>
+          <xacro:unless value="${use_body_length}">
+            <box size="${body_width} ${body_width} ${body_height}"/> <!-- [m] [m] [m] -->
+          </xacro:unless>
         </geometry>
       </collision>

File: rotors_description/urdf/neo11.xacro (robot description, xacro)
@@ -58,4 +58,6 @@
     robot_namespace="${namespace}"
     mass="${mass}"
+    use_body_length="false"
+    body_length=""
     body_width="${body_width}"
     body_height="${body_height}"

File: rotors_description/urdf/neo9.xacro (robot description, xacro)
@@ -58,4 +58,6 @@
     robot_namespace="${namespace}"
     mass="${mass}"
+    use_body_length="false"
+    body_length=""
     body_width="${body_width}"
     body_height="${body_height}"

File: rotors_description/urdf/pelican.xacro (robot description, xacro)
@@ -51,4 +51,6 @@
     robot_namespace="${namespace}"
     mass="${mass}"
+    use_body_length="false"
+    body_length=""
     body_width="${body_width}"
     body_height="${body_height}"

File: rotors_gazebo/models/rotors_description/urdf/iris.xacro (robot description, xacro)
@@ -46,4 +46,6 @@
     robot_namespace="${namespace}"
     mass="${mass}"
+    use_body_length="false"
+    body_length=""
     body_width="${body_width}"
     body_height="${body_height}"
