Commit message: movi el Cg a 0 0 0

File: rotors_description/urdf/multirotor_base.xacro (robot description, xacro)
@@ -43,5 +43,5 @@
       <inertial>
         <mass value="${mass}" />  <!-- [kg] -->
-        <origin xyz="0 0 -.05" />
+        <origin xyz="0 0 0" />
         <xacro:insert_block name="inertia" />
       </inertial>
