Commit message: cambie el orden de algunas variable spara separar las corroboradas

File: rotors_description/urdf/kamikaze.xacro (robot description, xacro)
@@ -5,14 +5,14 @@
   <!-- Properties -->
   <xacro:property name="namespace" value="$(arg namespace)" />
-  <xacro:property name="rotor_velocity_slowdown_sim" value="10" />
   <xacro:property name="use_mesh_file" value="true" />
   <xacro:property name="mesh_file" value="package://rotors_description/meshes/kamikaze.dae" />
-  <xacro:property name="mass" value="1.5" /> <!-- [kg] -->
   <xacro:property name="use_body_length" value="true" />
   <xacro:property name="body_length" value="1" />
-  <xacro:property name="body_width" value=".22" /> <!-- [m] --> <!-- FIXME: revisar -->
+  <xacro:property name="body_width" value=".22" /> <!-- [m] -->
   <xacro:property name="body_height" value="0.45" /> <!-- [m] -->
+  <!-- Properties TBC-->
+  <xacro:property name="rotor_velocity_slowdown_sim" value="10" />
+  <xacro:property name="mass" value="1.5" /> <!-- [kg] -->
   <xacro:property name="mass_rotor" value="0.005" /> <!-- [kg] -->
-  <xacro:property name="rotor_offset_top" value="0.037" /> <!-- [m] -->
   <xacro:property name="radius_rotor" value="0.1" /> <!-- [m] -->
   <xacro:property name="motor_constant" value="8.54858e-06" /> <!-- [kg m/s^2] -->

Commit message: nico te quiero mucho, espero que este año nos podamos egresar

File: rotors_description/urdf/kamikaze.xacro (robot description, xacro)
@@ -31,5 +31,5 @@
     <xacro:box_inertia x="${radius_rotor}" y="0.015" z="0.003" mass="${mass_rotor*rotor_velocity_slowdown_sim}" />
   </xacro:property>
-  <!-- Included URDF Files -->
+  <!-- Included URDF Motors Files -->
   <xacro:include filename="$(find rotors_description)/urdf/multirotor_base.xacro" />
   <!-- Instantiate multirotor_base_macro once -->
@@ -89,3 +89,75 @@
     <xacro:insert_block name="rotor_inertia" />
   </xacro:vertical_rotor>
+  <!-- modelo servo -->
+  <joint name="${namespace}/elevon_0_revolutejoint" type="continuous">
+    <axis xyz="1 0 0" />
+    <origin xyz="2 0 0.059" rpy="0 0 0" />
+    <parent link="${namespace}/base_link" />
+    <child link="${namespace}/tilt_unit_0" />
+  </joint>
+  <link name="${namespace}/tilt_unit_0">
+    <inertial>
+      <mass value="0.1" />
+      <xacro:insert_block name="body_inertia" />
+    </inertial>
+    <visual>
+      <geometry>
+        <box size="0.5 0.2 0.5"/>
+      </geometry>
+    </visual>
+    <collision>
+      <geometry>
+        <box size="0.005 0.005 0.005" />
+        <!-- [m] -->
+      </geometry>
+    </collision>
+  </link>
+  <gazebo>
+    <plugin name="right_tilt_unit_model" filename="librotors_gazebo_motor_model.so">
+      <robotNamespace>kamikaze</robotNamespace>
+      <jointName>kamikaze/tilt_unit_0_revolutejoint</jointName>
+      <linkName>kamikaze/tilt_unit_0</linkName>
+      <turningDirection>ccw</turningDirection>
+      <motorType>position</motorType>
+      <commandSubTopic>tilt_angle</commandSubTopic>
+      <motorNumber>2</motorNumber>
+      <motorSpeedPubTopic>tilt_motor_0/velocity</motorSpeedPubTopic>
+      <motorPositionPubTopic>tilt_motor_0/position</motorPositionPubTopic>
+      <joint_control_pid>
+        <p>1.0</p>
+        <i>0.0</i>
+        <d>0.01</d>
+        <iMax>1.0</iMax>
+        <iMin>-1.0</iMin>
+        <cmdMax>2.0</cmdMax>
+        <cmdMin>-2.0</cmdMin>
+      </joint_control_pid>
+    </plugin>
+  </gazebo>
+  <gazebo reference="${namespace}/tilt_unit_0">
+    <material>Gazebo/White</material>
+  </gazebo>
+  <!-- Elevon -->
+  <!-- <joint name="rotor_${motor_number}_joint" type="continuous">
+    <origin xyz="0 0 ${rotor_offset_top}" rpy="0 0 0" />
+    <axis xyz="0 0 1" />
+    <parent link="${namespace}/tilt_unit_${motor_number}" />
+    <child link="rotor_${motor_number}" />
+  </joint>
+  <link name="rotor_${motor_number}">
+    <inertial>
+      <mass value="${mass_rotor}" />
+      <xacro:insert_block name="inertia" />
+    </inertial>
+    <visual>
+      <geometry>
+        <mesh filename="package://rotors_description/meshes/${mesh}_${direction}.dae" scale="${radius_rotor} ${radius_rotor} ${radius_rotor}" />
+      </geometry>
+    </visual>
+    <collision>
+      <geometry>
+        <cylinder length="0.005" radius="${radius_rotor}" />
+      </geometry>
+    </collision>
+  </link> -->
 </robot>

Commit message: listos los topics de elevon

File: rotors_description/urdf/kamikaze.xacro (robot description, xacro)
@@ -90,11 +90,11 @@
   </xacro:vertical_rotor>
   <!-- modelo servo -->
-  <joint name="${namespace}/elevon_0_revolutejoint" type="continuous">
+  <joint name="${namespace}/elevon_2_revolutejoint" type="continuous">
     <axis xyz="1 0 0" />
     <origin xyz="2 0 0.059" rpy="0 0 0" />
     <parent link="${namespace}/base_link" />
-    <child link="${namespace}/tilt_unit_0" />
+    <child link="${namespace}/elevon_unit_2" />
   </joint>
-  <link name="${namespace}/tilt_unit_0">
+  <link name="${namespace}/elevon_unit_2">
     <inertial>
       <mass value="0.1" />
@@ -114,14 +114,14 @@
   </link>
   <gazebo>
-    <plugin name="right_tilt_unit_model" filename="librotors_gazebo_motor_model.so">
-      <robotNamespace>kamikaze</robotNamespace>
-      <jointName>kamikaze/tilt_unit_0_revolutejoint</jointName>
-      <linkName>kamikaze/tilt_unit_0</linkName>
+    <plugin name="elevon_unit_2_unit_model" filename="librotors_gazebo_motor_model.so">
+      <robotNamespace>${namespace}</robotNamespace>
+      <jointName>${namespace}/elevon_2_revolutejoint</jointName>
+      <linkName>${namespace}/elevon_unit_2</linkName>
       <turningDirection>ccw</turningDirection>
       <motorType>position</motorType>
-      <commandSubTopic>tilt_angle</commandSubTopic>
+      <commandSubTopic>command/elevon_2_angle</commandSubTopic>
       <motorNumber>2</motorNumber>
-      <motorSpeedPubTopic>tilt_motor_0/velocity</motorSpeedPubTopic>
-      <motorPositionPubTopic>tilt_motor_0/position</motorPositionPubTopic>
+      <motorSpeedPubTopic>elevon/2/velocity</motorSpeedPubTopic>
+      <motorPositionPubTopic>elevon/2/position</motorPositionPubTopic>
       <joint_control_pid>
         <p>1.0</p>
@@ -135,6 +135,6 @@
     </plugin>
   </gazebo>
-  <gazebo reference="${namespace}/tilt_unit_0">
-    <material>Gazebo/White</material>
+  <gazebo reference="${namespace}/elevon_unit_2">
+    <material>Gazebo/Red</material>
   </gazebo>
   <!-- Elevon -->

File: rotors_description/urdf/multirotor_base.xacro (robot description, xacro)
@@ -105,5 +105,5 @@
             <mesh filename="${mesh}"
               scale="1 1 1" />
-          </xacro:if>
+          </xacro:if>multirotor_base
           <xacro:unless value="${use_own_mesh}">
             <mesh filename="package://rotors_description/meshes/propeller_${direction}.dae"

File: rotors_description/urdf/overactuated_base.xacro (robot description, xacro)
@@ -67,7 +67,7 @@
       <axis xyz="1 0 0" />
       <parent link="${parent}" />
-      <child link="${namespace}/tilt_unit_${motor_number}" />
-    </joint>
-    <link name="${namespace}/tilt_unit_${motor_number}">
+      <child link="${robot_namespace}/tilt_unit_${motor_number}" />
+    </joint>
+    <link name="${robot_namespace}/tilt_unit_${motor_number}">
       <inertial>
         <mass value="${mass_tilt_unit}" /> <!-- [kg] -->
@@ -89,6 +89,6 @@
       <plugin name="${suffix}_tilt_unit_model" filename="librotors_gazebo_motor_model.so">
         <robotNamespace>${robot_namespace}</robotNamespace>
-        <jointName>${namespace}/tilt_unit_${motor_number}_revolutejoint</jointName>
-        <linkName>${namespace}/tilt_unit_${motor_number}</linkName>
+        <jointName>${robot_namespace}/tilt_unit_${motor_number}_revolutejoint</jointName>
+        <linkName>${robot_namespace}/tilt_unit_${motor_number}</linkName>
         <turningDirection>ccw</turningDirection>
         <motorType>position</motorType>
@@ -108,5 +108,5 @@
       </plugin>
     </gazebo>
-    <gazebo reference="${namespace}/tilt_unit_${motor_number}">
+    <gazebo reference="${robot_namespace}/tilt_unit_${motor_number}">
       <material>Gazebo/White</material>
     </gazebo>
@@ -115,5 +115,5 @@
       <origin xyz="0 0 ${rotor_offset_top}" rpy="0 0 0" />
       <axis xyz="0 0 1" />
-      <parent link="${namespace}/tilt_unit_${motor_number}" />
+      <parent link="${robot_namespace}/tilt_unit_${motor_number}" />
       <child link="rotor_${motor_number}" />
     </joint>
@@ -166,7 +166,7 @@
       <axis xyz="1 0 0" />
       <parent link="${parent}" />
-      <child link="${namespace}/tilt_unit_${motor_number}" />
-    </joint>
-    <link name="${namespace}/tilt_unit_${motor_number}">
+      <child link="${robot_namespace}/tilt_unit_${motor_number}" />
+    </joint>
+    <link name="${robot_namespace}/tilt_unit_${motor_number}">
       <inertial>
         <mass value="${mass_tilt_unit}" /> <!-- [kg] -->
@@ -207,6 +207,6 @@
       </plugin>
     </gazebo>
-    <gazebo reference="${namespace}/tilt_unit_${motor_number}">
-      <material>Gazebo/White</material>
+    <gazebo reference="${robot_namespace}/tilt_unit_${motor_number}">
+      <material>Gazebo/${color}</material>
     </gazebo>
     <!-- Upper Rotor -->
@@ -214,5 +214,5 @@
       <origin xyz="0 0 ${rotor_offset_top}" rpy="0 0 0" />
       <axis xyz="0 0 1" />
-      <parent link="${namespace}/tilt_unit_${motor_number}" />
+      <parent link="${robot_namespace}/tilt_unit_${motor_number}" />
       <child link="rotor_${motor_number}" />
     </joint>
@@ -260,5 +260,5 @@
       <origin xyz="0 0 ${-rotor_offset_top}" rpy="0 0 0" />
       <axis xyz="0 0 1" />
-      <parent link="${namespace}/tilt_unit_${motor_number}" />
+      <parent link="${robot_namespace}/tilt_unit_${motor_number}" />
       <child link="rotor_${motor_number+6}" />
     </joint>

Commit message: agregando segundo elevon

File: rotors_description/urdf/kamikaze.xacro (robot description, xacro)
@@ -92,5 +92,6 @@
   <joint name="${namespace}/elevon_2_revolutejoint" type="continuous">
     <axis xyz="1 0 0" />
-    <origin xyz="2 0 0.059" rpy="0 0 0" />
+    <property name="mesh_file" value="package://rotors_description/meshes/kamikaze.dae" />
+    <origin xyz="0.002 0 0.0008" rpy="0 0 0" />
     <parent link="${namespace}/base_link" />
     <child link="${namespace}/elevon_unit_2" />
@@ -103,5 +104,6 @@
     <visual>
       <geometry>
-        <box size="0.5 0.2 0.5"/>
+        <!-- <box size="0.5 0.2 0.5"/> -->
+        <mesh filename="package://rotors_description/meshes/elevon_left.dae"/>
       </geometry>
     </visual>
@@ -136,4 +138,55 @@
   </gazebo>
   <gazebo reference="${namespace}/elevon_unit_2">
+    <material>Gazebo/Blue</material>
+  </gazebo>
+  <!-- elevon 2 -->
+  <joint name="${namespace}/elevon_3_revolutejoint" type="continuous">
+    <axis xyz="1 0 0" />
+    <property name="mesh_file" value="package://rotors_description/meshes/kamikaze.dae" />
+    <!-- <origin xyz="-2 0.1 -0.8" rpy="0 0 0" /> -->
+    <parent link="${namespace}/base_link" />
+    <child link="${namespace}/elevon_unit_3"/>
+  </joint>
+  <link name="${namespace}/elevon_unit_3">
+    <inertial>
+      <mass value="0.1" />
+      <xacro:insert_block name="body_inertia" />
+    </inertial>
+    <visual>
+      <geometry>
+        <!-- <box size="0.5 0.2 0.5"/> -->
+        <mesh filename="package://rotors_description/meshes/elevon_rigth.dae"/>
+      </geometry>
+    </visual>
+    <collision>
+      <geometry>
+        <box size="0.005 0.005 0.005" />
+        <!-- [m] -->
+      </geometry>
+    </collision>
+  </link>
+  <gazebo>
+    <plugin name="elevon_unit_3_unit_model" filename="librotors_gazebo_motor_model.so">
+      <robotNamespace>${namespace}</robotNamespace>
+      <jointName>${namespace}/elevon_3_revolutejoint</jointName>
+      <linkName>${namespace}/elevon_unit_3</linkName>
+      <turningDirection>ccw</turningDirection>
+      <motorType>position</motorType>
+      <commandSubTopic>command/elevon_3_angle</commandSubTopic>
+      <motorNumber>3</motorNumber>
+      <motorSpeedPubTopic>elevon/3/velocity</motorSpeedPubTopic>
+      <motorPositionPubTopic>elevon/3/position</motorPositionPubTopic>
+      <joint_control_pid>
+        <p>0.5</p>
+        <i>0.5</i>
+        <d>0.1</d>
+        <iMax>1.0</iMax>
+        <iMin>-1.0</iMin>
+        <cmdMax>2.0</cmdMax>
+        <cmdMin>-2.0</cmdMin>
+      </joint_control_pid>
+    </plugin>
+  </gazebo>
+  <gazebo reference="${namespace}/elevon_unit_3">
     <material>Gazebo/Red</material>
   </gazebo>

Commit message: servos ok

File: rotors_description/urdf/kamikaze.xacro (robot description, xacro)
@@ -93,5 +93,5 @@
     <axis xyz="1 0 0" />
     <property name="mesh_file" value="package://rotors_description/meshes/kamikaze.dae" />
-    <origin xyz="0.002 0 0.0008" rpy="0 0 0" />
+    <origin xyz="0.11 0 -0.088" rpy="0 0.17 0" />
     <parent link="${namespace}/base_link" />
     <child link="${namespace}/elevon_unit_2" />
@@ -103,13 +103,14 @@
     </inertial>
     <visual>
-      <geometry>
-        <!-- <box size="0.5 0.2 0.5"/> -->
-        <mesh filename="package://rotors_description/meshes/elevon_left.dae"/>
+      <origin xyz="0.135 0 -0.0175" rpy="0 0 0" />
+      <geometry>
+        <box size="0.27 0.01 0.035"/>
+        <!-- <mesh filename="package://rotors_description/meshes/elevon_left.dae"/> -->
       </geometry>
     </visual>
     <collision>
-      <geometry>
-        <box size="0.005 0.005 0.005" />
-        <!-- [m] -->
+      <origin xyz="0.135 0 -0.0175" rpy="0 0 0" />
+      <geometry>
+        <box size="0.27 0.01 0.035"/>
       </geometry>
     </collision>
@@ -123,5 +124,5 @@
       <motorType>position</motorType>
       <commandSubTopic>command/elevon_2_angle</commandSubTopic>
-      <motorNumber>2</motorNumber>
+      <motorNumber>0</motorNumber>
       <motorSpeedPubTopic>elevon/2/velocity</motorSpeedPubTopic>
       <motorPositionPubTopic>elevon/2/position</motorPositionPubTopic>
@@ -144,5 +145,5 @@
     <axis xyz="1 0 0" />
     <property name="mesh_file" value="package://rotors_description/meshes/kamikaze.dae" />
-    <!-- <origin xyz="-2 0.1 -0.8" rpy="0 0 0" /> -->
+    <origin xyz="-0.11 0 -0.088" rpy="0 2.96 0" />
     <parent link="${namespace}/base_link" />
     <child link="${namespace}/elevon_unit_3"/>
@@ -154,15 +155,16 @@
     </inertial>
     <visual>
-      <geometry>
-        <!-- <box size="0.5 0.2 0.5"/> -->
-        <mesh filename="package://rotors_description/meshes/elevon_rigth.dae"/>
-      </geometry>
-    </visual>
-    <collision>
-      <geometry>
-        <box size="0.005 0.005 0.005" />
-        <!-- [m] -->
-      </geometry>
-    </collision>
+        <origin xyz="0.135 0 0.0175" rpy="0 0 0" />
+        <geometry>
+          <box size="0.27 0.01 0.035"/>
+          <!-- <mesh filename="package://rotors_description/meshes/elevon_left.dae"/> -->
+        </geometry>
+      </visual>
+      <collision>
+        <origin xyz="-0.135 0 -0.0175" rpy="0 0 0" />
+        <geometry>
+          <box size="0.27 0.01 0.035"/>
+        </geometry>
+      </collision>
   </link>
   <gazebo>
@@ -174,5 +176,5 @@
       <motorType>position</motorType>
       <commandSubTopic>command/elevon_3_angle</commandSubTopic>
-      <motorNumber>3</motorNumber>
+      <motorNumber>1</motorNumber>
       <motorSpeedPubTopic>elevon/3/velocity</motorSpeedPubTopic>
       <motorPositionPubTopic>elevon/3/position</motorPositionPubTopic>

Commit message: pequena actualizacion del xacro

File: rotors_description/urdf/kamikaze.xacro (robot description, xacro)
@@ -20,5 +20,5 @@
   <xacro:property name="time_constant_up" value="0.0125" /> <!-- [s] -->
   <xacro:property name="time_constant_down" value="0.025" /> <!-- [s] -->
-  <xacro:property name="max_rot_velocity" value="838" /> <!-- [rad/s] -->
+  <xacro:property name="max_rot_velocity" value="1838" /> <!-- [rad/s] -->
   <xacro:property name="rotor_drag_coefficient" value="8.06428e-05" />
   <xacro:property name="rolling_moment_coefficient" value="0.000001" />
@@ -190,4 +190,22 @@
     </plugin>
   </gazebo>
+  <gazebo>
+    <plugin name="wing_0" filename="3libLiftDragPlugin.so">
+      <a0>0.0</a0>
+      <cla>4.752798721</cla>
+      <cda>0.6417112299</cda>
+      <cma>-1.8</cma>
+      <alpha_stall>0.3391428111</alpha_stall>
+      <cla_stall>-3.85</cla_stall>
+      <cda_stall>-0.9233984055</cda_stall>
+      <cma_stall>0</cma_stall>
+      <cp>-0.1 0 -0.5</cp>
+      <area>0.05</area>
+      <air_density>1.2041</air_density>
+      <forward>0 0 1</forward>
+      <upward>0 1 0</upward>
+      <link_name>${namespace}/base_link</link_name>
+    </plugin>
+  </gazebo>
   <gazebo reference="${namespace}/elevon_unit_3">
     <material>Gazebo/Red</material>

Commit message: agregue las variables aerodinamicas y la descripcion del otro ala

File: rotors_description/urdf/kamikaze.xacro (robot description, xacro)
@@ -23,4 +23,18 @@
   <xacro:property name="rotor_drag_coefficient" value="8.06428e-05" />
   <xacro:property name="rolling_moment_coefficient" value="0.000001" />
+  <!-- Aerodynamics -->
+  <!-- Henry's -->
+  <xacro:property name="ao"           value="-0.0131" />
+  <xacro:property name="cla"          value="6.4983" />
+  <xacro:property name="alpha_stall"  value="0.284" />
+  <xacro:property name="cla_stall"    value="-3.8268" />
+  <xacro:property name="area"         value="0.040132" /> <!-- in m^2, dont know if its ok -->
+  <!-- World -->
+  <xacro:property name="air_density"  value="1.2041" />
+  <!-- TBC - this parameters are from plane.sdf -->
+  <xacro:property name="cda"          value="0.6417112299" />
+  <xacro:property name="cma"          value="-1.8" />
+  <xacro:property name="cda_stall"    value="-0.9233984055" />
+  <xacro:property name="cma_stall"    value="0.0" />
   <!-- Property Blocks -->
   <xacro:property name="body_inertia">
@@ -168,4 +182,7 @@
       </collision>
   </link>
+  <gazebo reference="${namespace}/elevon_unit_3">
+    <material>Gazebo/Red</material>
+  </gazebo>
   <gazebo>
     <plugin name="elevon_unit_3_unit_model" filename="librotors_gazebo_motor_model.so">
@@ -190,22 +207,23 @@
     </plugin>
   </gazebo>
+  <!-- liftDrag 1 -->
   <gazebo>
     <plugin name="wing_0" filename="libLiftDragPlugin.so">
-      <a0>0.0</a0>
-      <cla>4.752798721</cla>
-      <cda>0.6417112299</cda>
-      <cma>-1.8</cma>
-      <alpha_stall>0.3391428111</alpha_stall>
-      <cla_stall>-3.85</cla_stall>
-      <cda_stall>-0.9233984055</cda_stall>
-      <cma_stall>0</cma_stall>
-      <cp>-0.1 0 -0.5</cp>
-      <area>0.05</area>
-      <air_density>1.2041</air_density>
+      <a0>${a0}</a0>
+      <cla>${cla}</cla>
+      <cda>${cda}</cda>
+      <cma>${cma}</cma>
+      <alpha_stall>${alpha_stall}</alpha_stall>
+      <cla_stall>${cla_stall}</cla_stall>
+      <cda_stall>${cda_stall}</cda_stall>
+      <cma_stall>${cma_stall}</cma_stall>
+      <cp>-0.1 0 -0.5</cp><!-- FIXME!!!! -->
+      <area>${area}</area>
+      <air_density>${air_density}</air_density>
       <forward>0 0 1</forward>
       <upward>0 1 0</upward>
       <link_name>${namespace}/base_link</link_name>
       <control_joint_name>${namespace}/elevon_2_revolutejoint</control_joint_name>
-      <control_joint_rad_to_cl>-0.5</control_joint_rad_to_cl>
+      <control_joint_rad_to_cl>${control_joint_rad_to_cl}</control_joint_rad_to_cl>
       <velocity_joint_name>${namespace}/rotor_0_joint</velocity_joint_name>
       <rotorVelocitySlowdownSim>${rotor_velocity_slowdown_sim}</rotorVelocitySlowdownSim>
@@ -213,29 +231,27 @@
     </plugin>
   </gazebo>
-  <gazebo reference="${namespace}/elevon_unit_3">
-    <material>Gazebo/Red</material>
-  </gazebo>
-  <!-- Elevon -->
-  <!-- <joint name="rotor_${motor_number}_joint" type="continuous">
-    <origin xyz="0 0 ${rotor_offset_top}" rpy="0 0 0" />
-    <axis xyz="0 0 1" />
-    <parent link="${namespace}/tilt_unit_${motor_number}" />
-    <child link="rotor_${motor_number}" />
-  </joint>
-  <link name="rotor_${motor_number}">
-    <inertial>
-      <mass value="${mass_rotor}" />
-      <xacro:insert_block name="inertia" />
-    </inertial>
-    <visual>
-      <geometry>
-        <mesh filename="package://rotors_description/meshes/${mesh}_${direction}.dae" scale="${radius_rotor} ${radius_rotor} ${radius_rotor}" />
-      </geometry>
-    </visual>
-    <collision>
-      <geometry>
-        <cylinder length="0.005" radius="${radius_rotor}" />
-      </geometry>
-    </collision>
-  </link> -->
+  <!-- liftDrag 2 -->
+  <gazebo>
+    <plugin name="wing_1" filename="libLiftDragPlugin.so">
+      <a0>${a0}</a0>
+      <cla>${cla}</cla>
+      <cda>${cda}</cda>
+      <cma>${cma}</cma>
+      <alpha_stall>${alpha_stall}</alpha_stall>
+      <cla_stall>${cla_stall}</cla_stall>
+      <cda_stall>${cda_stall}</cda_stall>
+      <cma_stall>${cma_stall}</cma_stall>
+      <cp>-0.1 0 -0.5</cp><!-- FIXME!!!! -->
+      <area>${area}</area>
+      <air_density>${air_density}</air_density>
+      <forward>0 0 1</forward>
+      <upward>0 1 0</upward>
+      <link_name>${namespace}/base_link</link_name>
+      <control_joint_name>${namespace}/elevon_3_revolutejoint</control_joint_name>
+      <control_joint_rad_to_cl>${control_joint_rad_to_cl}</control_joint_rad_to_cl>
+      <velocity_joint_name>${namespace}/rotor_1_joint</velocity_joint_name>
+      <rotorVelocitySlowdownSim>${rotor_velocity_slowdown_sim}</rotorVelocitySlowdownSim>
+      <motorConstant>${motor_constant}</motorConstant>
+    </plugin>
+  </gazebo>
 </robot>

Commit message: dos typos

File: rotors_description/urdf/kamikaze.xacro (robot description, xacro)
@@ -25,5 +25,5 @@
   <!-- Aerodynamics -->
   <!-- Henry's -->
-  <xacro:property name="ao"           value="-0.0131" />
+  <xacro:property name="a0"           value="-0.0131" />
   <xacro:property name="cla"          value="6.4983" />
   <xacro:property name="alpha_stall"  value="0.284" />
@@ -37,4 +37,5 @@
   <xacro:property name="cda_stall"    value="-0.9233984055" />
   <xacro:property name="cma_stall"    value="0.0" />
+  <xacro:property name="control_joint_rad_to_cl"    value="-0.5" />
   <!-- Property Blocks -->
   <xacro:property name="body_inertia">

Commit message: Borre algunos espacios y lineas en blanco, un mesh que no usabamos y cambie la masa de los elevones

File: rotors_description/urdf/kamikaze.xacro (robot description, xacro)
@@ -1,5 +1,3 @@
 <?xml version="1.0"?>
-<!--
--->
 <robot name="kamikaze" xmlns:xacro="http://ros.org/wiki/xacro">
   <!-- Properties -->
@@ -114,5 +112,5 @@
   <link name="${namespace}/elevon_unit_2">
     <inertial>
-      <mass value="0.1" />
+      <mass value="0.01" />
       <xacro:insert_block name="body_inertia" />
     </inertial>
@@ -121,5 +119,4 @@
       <geometry>
         <box size="0.27 0.01 0.035"/>
-        <!-- <mesh filename="package://rotors_description/meshes/elevon_left.dae"/> -->
       </geometry>
     </visual>
@@ -166,5 +163,5 @@
   <link name="${namespace}/elevon_unit_3">
     <inertial>
-      <mass value="0.1" />
+      <mass value="0.01" />
       <xacro:insert_block name="body_inertia" />
     </inertial>
