Commit message: pareceria ser estable esta config, si achico los parametros de inercia explota la simulacion

File: rotors_description/urdf/kamikaze.xacro (robot description, xacro)
@@ -39,4 +39,7 @@
   <xacro:property name="body_inertia">
     <inertia ixx="0.006" ixy="0.0" ixz="0.0" iyy="0.074" iyz="0.0" izz="0.069" /> <!-- [kg m^2] [kg m^2] [kg m^2] [kg m^2] [kg m^2] [kg m^2] -->
+  </xacro:property>
+  <xacro:property name="elevon_inertia">
+    <inertia ixx="0.001" ixy="0.0" ixz="0.0" iyy="0.001" iyz="0.0" izz="0.001" /> <!-- [kg m^2] [kg m^2] [kg m^2] [kg m^2] [kg m^2] [kg m^2] -->
   </xacro:property>
   <!-- inertia of a single rotor, assuming it is a cuboid. Height=3mm, width=15mm -->
@@ -113,5 +116,5 @@
     <inertial>
       <mass value="0.01" />
-      <xacro:insert_block name="body_inertia" />
+      <xacro:insert_block name="elevon_inertia" />
     </inertial>
     <visual>
@@ -164,5 +167,5 @@
     <inertial>
       <mass value="0.01" />
-      <xacro:insert_block name="body_inertia" />
+      <xacro:insert_block name="elevon_inertia" />
     </inertial>
     <visual>
@@ -170,5 +173,4 @@
         <geometry>
           <box size="0.27 0.01 0.035"/>
-          <!-- <mesh filename="package://rotors_description/meshes/elevon_left.dae"/> -->
         </geometry>
       </visual>

Commit message: separe las properties en un archivo aparte asi es mas facil de leer

File: rotors_description/urdf/kamikaze.xacro (robot description, xacro)
@@ -1,50 +1,6 @@
 <?xml version="1.0"?>
 <robot name="kamikaze" xmlns:xacro="http://ros.org/wiki/xacro">
-  <!-- Properties -->
-  <xacro:property name="namespace" value="$(arg namespace)" />
-  <xacro:property name="use_mesh_file" value="true" />
-  <xacro:property name="mesh_file" value="package://rotors_description/meshes/kamikaze.dae" />
-  <xacro:property name="use_body_length" value="true" />
-  <xacro:property name="body_length" value="1" />
-  <xacro:property name="body_width" value=".22" /> <!-- [m] -->
-  <xacro:property name="body_height" value="0.45" /> <!-- [m] -->
-  <!-- Properties TBC-->
-  <xacro:property name="rotor_velocity_slowdown_sim" value="10" />
-  <xacro:property name="mass" value="1.5" /> <!-- [kg] -->
-  <xacro:property name="mass_rotor" value="0.005" /> <!-- [kg] -->
-  <xacro:property name="radius_rotor" value="0.1" /> <!-- [m] -->
-  <xacro:property name="motor_constant" value="8.54858e-06" /> <!-- [kg m/s^2] -->
-  <xacro:property name="moment_constant" value="0.016" /> <!-- [m] -->
-  <xacro:property name="time_constant_up" value="0.0125" /> <!-- [s] -->
-  <xacro:property name="time_constant_down" value="0.025" /> <!-- [s] -->
-  <xacro:property name="max_rot_velocity" value="1838" /> <!-- [rad/s] -->
-  <xacro:property name="rotor_drag_coefficient" value="8.06428e-05" />
-  <xacro:property name="rolling_moment_coefficient" value="0.000001" />
-  <!-- Aerodynamics -->
-  <!-- Henry's -->
-  <xacro:property name="a0"           value="-0.0131" />
-  <xacro:property name="cla"          value="6.4983" />
-  <xacro:property name="alpha_stall"  value="0.284" />
-  <xacro:property name="cla_stall"    value="-3.8268" />
-  <xacro:property name="area"         value="0.040132" /> <!-- in m^2, dont know if its ok -->
-  <!-- World -->
-  <xacro:property name="air_density"  value="1.2041" />
-  <!-- TBC - this parameters are from plane.sdf -->
-  <xacro:property name="cda"          value="0.6417112299" />
-  <xacro:property name="cma"          value="-1.8" />
-  <xacro:property name="cda_stall"    value="-0.9233984055" />
-  <xacro:property name="cma_stall"    value="0.0" />
-  <xacro:property name="control_joint_rad_to_cl"    value="-0.5" />
-  <!-- Property Blocks -->
-  <xacro:property name="body_inertia">
-    <inertia ixx="0.006" ixy="0.0" ixz="0.0" iyy="0.074" iyz="0.0" izz="0.069" /> <!-- [kg m^2] [kg m^2] [kg m^2] [kg m^2] [kg m^2] [kg m^2] -->
-  </xacro:property>
-  <xacro:property name="elevon_inertia">
-    <inertia ixx="0.001" ixy="0.0" ixz="0.0" iyy="0.001" iyz="0.0" izz="0.001" /> <!-- [kg m^2] [kg m^2] [kg m^2] [kg m^2] [kg m^2] [kg m^2] -->
-  </xacro:property>
-  <!-- inertia of a single rotor, assuming it is a cuboid. Height=3mm, width=15mm -->
-  <xacro:property name="rotor_inertia">
-    <xacro:box_inertia x="${radius_rotor}" y="0.015" z="0.003" mass="${mass_rotor*rotor_velocity_slowdown_sim}" />
-  </xacro:property>
+  <!-- Included URDF Motors Files -->
+  <xacro:include filename="$(find rotors_description)/urdf/kamikaze_properties.xacro" />
   <!-- Included URDF Motors Files -->
   <xacro:include filename="$(find rotors_description)/urdf/multirotor_base.xacro" />

Commit message: commit con anclaje en z

File: rotors_description/urdf/kamikaze.xacro (robot description, xacro)
@@ -1,4 +1,5 @@
 <?xml version="1.0"?>
 <robot name="kamikaze" xmlns:xacro="http://ros.org/wiki/xacro">
+  <link name="world"/>
   <!-- Included URDF Motors Files -->
   <xacro:include filename="$(find rotors_description)/urdf/kamikaze_properties.xacro" />
@@ -165,5 +166,5 @@
   <!-- liftDrag 1 -->
   <gazebo>
-    <plugin name="wing_0" filename="libLiftDragPlugin.so">
+    <plugin name="wing_0" filename="/home/sheila/ros_sim/ros_ws/devel/lib/libLiftDragPlugin.so">
       <a0>${a0}</a0>
       <cla>${cla}</cla>
@@ -189,5 +190,5 @@
   <!-- liftDrag 2 -->
   <gazebo>
-    <plugin name="wing_1" filename="libLiftDragPlugin.so">
+    <plugin name="wing_1" filename="/home/sheila/ros_sim/ros_ws/devel/lib/libLiftDragPlugin.so">
       <a0>${a0}</a0>
       <cla>${cla}</cla>
@@ -211,3 +212,9 @@
     </plugin>
   </gazebo>
+  <joint name="world_fixed" type="continuous">
+     <parent link="world"/>
+     <child link="${namespace}/base_link"/>
+     <axis xyz="0 0 1" />
+     <origin xyz="0 0 1" rpy="0 0 0" />
+  </joint>
 </robot>

File: rotors_description/urdf/kamikaze_properties.xacro (robot description, xacro)
@@ -39,5 +39,5 @@
   <xacro:property name="cda_stall"    value="-0.9233984055" />
   <xacro:property name="cma_stall"    value="0.0" />
-  <xacro:property name="control_joint_rad_to_cl"    value="-0.5" />
+  <xacro:property name="control_joint_rad_to_cl"    value="-1.5" />
   <!-- Property Blocks -->
   <xacro:property name="body_inertia">

Commit message: agregue una esfera en el CoG y ahi puse el joint ocn el mundo

File: rotors_description/urdf/kamikaze.xacro (robot description, xacro)
@@ -212,9 +212,30 @@
     </plugin>
   </gazebo>
+  <link name="esfera">
+    <inertial>
+      <mass value="0.0000001" /> <!-- [kg] -->
+      <xacro:insert_block name="elevon_inertia" />
+    </inertial>
+    <visual>
+      <geometry>
+        <sphere radius="0.05" />
+      </geometry>
+    </visual>
+  </link>
+  <gazebo reference="esfera">
+    <material>Gazebo/Green</material>
+  </gazebo>
   <joint name="world_fixed" type="continuous">
      <parent link="world"/>
-     <child link="${namespace}/base_link"/>
-     <axis xyz="0 0 1" />
+     <child link="esfera"/>
+     <axis xyz="1 0 0" />
      <origin xyz="0 0 1" rpy="0 0 0" />
   </joint>
+  <joint name="CoG" type="fixed">
+    <origin xyz="0 0 .05" rpy="0 0 0" />
+    <child link="${namespace}/base_link"/>
+    <parent link="esfera"/>
+    <!-- <axis xyz="1 0 0" /> -->
+    <!-- <origin xyz="0 0 1" rpy="0 0 0" /> -->
+  </joint>
 </robot>

File: rotors_description/urdf/kamikaze_properties.xacro (robot description, xacro)
@@ -39,5 +39,5 @@
   <xacro:property name="cda_stall"    value="-0.9233984055" />
   <xacro:property name="cma_stall"    value="0.0" />
-  <xacro:property name="control_joint_rad_to_cl"    value="-1.5" />
+  <xacro:property name="control_joint_rad_to_cl"    value="-0.5" />
   <!-- Property Blocks -->
   <xacro:property name="body_inertia">

File: rotors_description/urdf/multirotor_base.xacro (robot description, xacro)
@@ -43,5 +43,5 @@
       <inertial>
         <mass value="${mass}" />  <!-- [kg] -->
-        <origin xyz="0 0 0" />
+        <origin xyz="0 0 -.05" />
         <xacro:insert_block name="inertia" />
       </inertial>

Commit message: revisando eje x

File: rotors_description/urdf/kamikaze.xacro (robot description, xacro)
@@ -166,5 +166,5 @@
   <!-- liftDrag 1 -->
   <gazebo>
-    <plugin name="wing_0" filename="/home/sheila/ros_sim/ros_ws/devel/lib/libLiftDragPlugin.so">
+    <plugin name="wing_0" filename="/home/pablo/Documentos/UTN/proyecto/ros_sim/ros_ws/devel/lib/libLiftDragPlugin.so">
       <a0>${a0}</a0>
       <cla>${cla}</cla>
@@ -190,5 +190,5 @@
   <!-- liftDrag 2 -->
   <gazebo>
-    <plugin name="wing_1" filename="/home/sheila/ros_sim/ros_ws/devel/lib/libLiftDragPlugin.so">
+    <plugin name="wing_1" filename="/home/pablo/Documentos/UTN/proyecto/ros_sim/ros_ws/devel/lib/libLiftDragPlugin.so">
       <a0>${a0}</a0>
       <cla>${cla}</cla>
@@ -214,5 +214,5 @@
   <link name="esfera">
     <inertial>
-      <mass value="0.0000001" /> <!-- [kg] -->
+      <mass value="0.0000001" />
       <xacro:insert_block name="elevon_inertia" />
     </inertial>
@@ -223,19 +223,40 @@
     </visual>
   </link>
-  <gazebo reference="esfera">
+   <gazebo reference="esfera">
     <material>Gazebo/Green</material>
   </gazebo>
-  <joint name="world_fixed" type="continuous">
+<!-- Control de altura -->
+<joint name="world_fixed" type="prismatic">
+  <parent link="world"/>
+  <child link="esfera"/>
+  <axis xyz="0 0 1" />
+  <origin xyz="0 0 1" rpy="0 0 0" />
+  <limit lower="0" upper="50" effort="20000" velocity="20000"/>
+</joint>
+<!-- Control de roll -->
+  <!-- <joint name="world_fixed" type="continuous">
+    <parent link="world"/>
+    <child link="esfera"/>
+    <axis xyz="0 1 0" />
+    <origin xyz="0 0 1" rpy="0 0 0" />
+  </joint> -->
+<!-- Control de pitch -->
+  <!-- <joint name="world_fixed" type="continuous">
      <parent link="world"/>
      <child link="esfera"/>
      <axis xyz="1 0 0" />
      <origin xyz="0 0 1" rpy="0 0 0" />
-  </joint>
+  </joint> -->
+<!-- Contro de yaw -->
+  <!-- <joint name="world_fixed" type="continuous">
+    <parent link="world"/>
+    <child link="${namespace}/base_link"/>
+    <axis xyz="0 0 1" />
+    <origin xyz="0 0 1" rpy="0 0 0" />
+  </joint> -->
   <joint name="CoG" type="fixed">
     <origin xyz="0 0 .05" rpy="0 0 0" />
     <child link="${namespace}/base_link"/>
     <parent link="esfera"/>
-    <!-- <axis xyz="1 0 0" /> -->
-    <!-- <origin xyz="0 0 1" rpy="0 0 0" /> -->
   </joint>
 </robot>

Commit message: deje los 4 ejes

File: rotors_description/urdf/kamikaze.xacro (robot description, xacro)
@@ -231,8 +231,40 @@
   <child link="esfera"/>
   <axis xyz="0 0 1" />
+  <origin xyz="0 0 0" rpy="0 0 0" />
+  <limit lower="0" upper="50" effort="20000" velocity="20000"/>
+</joint>
+<joint name="CoG" type="fixed">
+  <child link="${namespace}/base_link"/>
+  <parent link="esfera"/>
+  <origin xyz="0 0 .05" rpy="0 0 0" />
+  <axis xyz="0 0 1" />
+</joint>
+<!--  Control de Yaw-->
+<!-- <joint name="world_fixed" type="continuous">
+  <parent link="world"/>
+  <child link="esfera"/>
+  <axis xyz="0 0 1" />
   <origin xyz="0 0 1" rpy="0 0 0" />
-  <limit lower="0" upper="50" effort="20000" velocity="20000"/>
-</joint>
-<!-- Control de roll -->
+</joint>
+<joint name="CoG" type="fixed">
+  <child link="${namespace}/base_link"/>
+  <parent link="esfera"/>
+  <origin xyz="0 0 .05" rpy="0 0 0" />
+  <axis xyz="0 0 1" />
+</joint> -->
+<!-- Control de pitch -->
+<!-- <joint name="world_fixed" type="continuous">
+  <parent link="world"/>
+  <child link="esfera"/>
+  <axis xyz="1 0 0" />
+  <origin xyz="0 0 1" rpy="0 0 0" />
+</joint>
+<joint name="CoG" type="fixed">
+  <child link="${namespace}/base_link"/>
+  <parent link="esfera"/>
+  <origin xyz="0 0 .05" rpy="0 0 0" />
+  <axis xyz="1 0 0" />
+</joint> -->
+<!-- Contro de Roll -->
   <!-- <joint name="world_fixed" type="continuous">
     <parent link="world"/>
@@ -240,23 +272,11 @@
     <axis xyz="0 1 0" />
     <origin xyz="0 0 1" rpy="0 0 0" />
-  </joint> -->
-<!-- Control de pitch -->
-  <!-- <joint name="world_fixed" type="continuous">
-     <parent link="world"/>
-     <child link="esfera"/>
-     <axis xyz="1 0 0" />
-     <origin xyz="0 0 1" rpy="0 0 0" />
-  </joint> -->
-<!-- Contro de yaw -->
-  <!-- <joint name="world_fixed" type="continuous">
-    <parent link="world"/>
-    <child link="${namespace}/base_link"/>
-    <axis xyz="0 0 1" />
-    <origin xyz="0 0 1" rpy="0 0 0" />
-  </joint> -->
+  </joint>
   <joint name="CoG" type="fixed">
-    <origin xyz="0 0 .05" rpy="0 0 0" />
     <child link="${namespace}/base_link"/>
     <parent link="esfera"/>
-  </joint>
+    <origin xyz="0 0 .05" rpy="0 0 0" />
+    <axis xyz="0 1 0" />
+  </joint>
+ -->
 </robot>

Commit message: variando parametros motor

File: rotors_description/urdf/kamikaze.xacro (robot description, xacro)
@@ -1,5 +1,5 @@
 <?xml version="1.0"?>
 <robot name="kamikaze" xmlns:xacro="http://ros.org/wiki/xacro">
-  <link name="world"/>
+  <!-- <link name="world"/> -->
   <!-- Included URDF Motors Files -->
   <xacro:include filename="$(find rotors_description)/urdf/kamikaze_properties.xacro" />
@@ -178,7 +178,8 @@
       <area>${area}</area>
       <air_density>${air_density}</air_density>
-      <forward>0 0 1</forward>
+      <forward>0 0 -1</forward>
       <upward>0 1 0</upward>
-      <link_name>${namespace}/base_link</link_name>
+     <!-- <link_name>${namespace}/base_link</link_name> -->
+      <link_name>esfera</link_name>
       <control_joint_name>${namespace}/elevon_3_revolutejoint</control_joint_name>
       <control_joint_rad_to_cl>${control_joint_rad_to_cl}</control_joint_rad_to_cl>
@@ -204,5 +205,6 @@
       <forward>0 0 1</forward>
       <upward>0 1 0</upward>
-      <link_name>${namespace}/base_link</link_name>
+      <!-- <link_name>${namespace}/base_link</link_name> -->
+      <link_name>esfera</link_name>
       <control_joint_name>${namespace}/elevon_2_revolutejoint</control_joint_name>
       <control_joint_rad_to_cl>${control_joint_rad_to_cl}</control_joint_rad_to_cl>
@@ -212,5 +214,5 @@
     </plugin>
   </gazebo>
-  <link name="esfera">
+<!-- <link name="esfera">
     <inertial>
       <mass value="0.0000001" />
@@ -219,5 +221,5 @@
     <visual>
       <geometry>
-        <sphere radius="0.05" />
+        <sphere radius="0.005" />
       </geometry>
     </visual>
@@ -225,7 +227,7 @@
    <gazebo reference="esfera">
     <material>Gazebo/Green</material>
-  </gazebo>
+  </gazebo> -->
 <!-- Control de altura -->
-<joint name="world_fixed" type="prismatic">
+<!-- <joint name="world_fixed" type="prismatic">
   <parent link="world"/>
   <child link="esfera"/>
@@ -239,5 +241,5 @@
   <origin xyz="0 0 .05" rpy="0 0 0" />
   <axis xyz="0 0 1" />
-</joint>
+</joint> -->
 <!--  Control de Yaw-->
 <!-- <joint name="world_fixed" type="continuous">
@@ -278,5 +280,4 @@
     <origin xyz="0 0 .05" rpy="0 0 0" />
     <axis xyz="0 1 0" />
-  </joint>
- -->
+  </joint> -->
 </robot>

File: rotors_description/urdf/kamikaze_properties.xacro (robot description, xacro)
@@ -20,6 +20,6 @@
   <xacro:property name="motor_constant" value="8.54858e-06" /> <!-- [kg m/s^2] -->
   <xacro:property name="moment_constant" value="0.016" /> <!-- [m] -->
-  <xacro:property name="time_constant_up" value="0.0125" /> <!-- [s] -->
-  <xacro:property name="time_constant_down" value="0.025" /> <!-- [s] -->
+  <xacro:property name="time_constant_up" value= "0.0125" /> <!-- [s]  0125  125 -->
+  <xacro:property name="time_constant_down" value="0.025" /> <!-- [s]  025    25-->
   <xacro:property name="max_rot_velocity" value="1838" /> <!-- [rad/s] -->
   <xacro:property name="rotor_drag_coefficient" value="8.06428e-05" />

Commit message: calibrando yaw

File: rotors_description/urdf/kamikaze.xacro (robot description, xacro)
@@ -1,5 +1,5 @@
 <?xml version="1.0"?>
 <robot name="kamikaze" xmlns:xacro="http://ros.org/wiki/xacro">
-  <!-- <link name="world"/> -->
+  <link name="world"/>
   <!-- Included URDF Motors Files -->
   <xacro:include filename="$(find rotors_description)/urdf/kamikaze_properties.xacro" />
@@ -214,5 +214,5 @@
     </plugin>
   </gazebo>
-<!-- <link name="esfera">
+<link name="esfera">
     <inertial>
       <mass value="0.0000001" />
@@ -227,5 +227,5 @@
    <gazebo reference="esfera">
     <material>Gazebo/Green</material>
-  </gazebo> -->
+  </gazebo>
 <!-- Control de altura -->
 <!-- <joint name="world_fixed" type="prismatic">
@@ -243,5 +243,5 @@
 </joint> -->
 <!--  Control de Yaw-->
-<!-- <joint name="world_fixed" type="continuous">
+<joint name="world_fixed" type="continuous">
   <parent link="world"/>
   <child link="esfera"/>
@@ -254,5 +254,5 @@
   <origin xyz="0 0 .05" rpy="0 0 0" />
   <axis xyz="0 0 1" />
-</joint> -->
+</joint>
 <!-- Control de pitch -->
 <!-- <joint name="world_fixed" type="continuous">

Commit message: agregue un archivo para modificar el path de la lib

File: rotors_description/urdf/kamikaze.xacro (robot description, xacro)
@@ -2,5 +2,7 @@
 <robot name="kamikaze" xmlns:xacro="http://ros.org/wiki/xacro">
   <link name="world"/>
-  <!-- Included URDF Motors Files -->
+  <!-- Included URDF kamikaze properties -->
+  <xacro:include filename="$(find rotors_description)/urdf/kamikaze_liftDrag_path.xacro" />
+  <!-- Included URDF kamikaze properties -->
   <xacro:include filename="$(find rotors_description)/urdf/kamikaze_properties.xacro" />
   <!-- Included URDF Motors Files -->
@@ -65,5 +67,5 @@
   <joint name="${namespace}/elevon_2_revolutejoint" type="continuous">
     <axis xyz="1 0 0" />
-    <property name="mesh_file" value="package://rotors_description/meshes/kamikaze.dae" />
+    <xacro:property name="mesh_file" value="package://rotors_description/meshes/kamikaze.dae" />
     <origin xyz="0.11 0 -0.088" rpy="0 0.17 0" />
     <parent link="${namespace}/base_link" />
@@ -116,5 +118,5 @@
   <joint name="${namespace}/elevon_3_revolutejoint" type="continuous">
     <axis xyz="1 0 0" />
-    <property name="mesh_file" value="package://rotors_description/meshes/kamikaze.dae" />
+    <xacro:property name="mesh_file" value="package://rotors_description/meshes/kamikaze.dae" />
     <origin xyz="-0.11 0 -0.088" rpy="0 2.96 0" />
     <parent link="${namespace}/base_link" />
@@ -166,5 +168,5 @@
   <!-- liftDrag 1 -->
   <gazebo>
-    <plugin name="wing_0" filename="/home/pablo/Documentos/UTN/proyecto/ros_sim/ros_ws/devel/lib/libLiftDragPlugin.so">
+    <plugin name="wing_0" filename="${liftDragPath}/libLiftDragPlugin.so">
       <a0>${a0}</a0>
       <cla>${cla}</cla>
@@ -191,5 +193,5 @@
   <!-- liftDrag 2 -->
   <gazebo>
-    <plugin name="wing_1" filename="/home/pablo/Documentos/UTN/proyecto/ros_sim/ros_ws/devel/lib/libLiftDragPlugin.so">
+    <plugin name="wing_1" filename="${liftDragPath}/libLiftDragPlugin.so">
       <a0>${a0}</a0>
       <cla>${cla}</cla>

Commit message: Borre la esfera, ya no la necesitamos

File: rotors_description/urdf/kamikaze.xacro (robot description, xacro)
@@ -182,6 +182,5 @@
       <forward>0 0 -1</forward>
       <upward>0 1 0</upward>
-     <!-- <link_name>${namespace}/base_link</link_name> -->
-      <link_name>esfera</link_name>
+      <link_name>${namespace}/base_link</link_name>
       <control_joint_name>${namespace}/elevon_3_revolutejoint</control_joint_name>
       <control_joint_rad_to_cl>${control_joint_rad_to_cl}</control_joint_rad_to_cl>
@@ -207,6 +206,5 @@
       <forward>0 0 1</forward>
       <upward>0 1 0</upward>
-      <!-- <link_name>${namespace}/base_link</link_name> -->
-      <link_name>esfera</link_name>
+      <link_name>${namespace}/base_link</link_name>
       <control_joint_name>${namespace}/elevon_2_revolutejoint</control_joint_name>
       <control_joint_rad_to_cl>${control_joint_rad_to_cl}</control_joint_rad_to_cl>
@@ -216,70 +214,32 @@
     </plugin>
   </gazebo>
-<link name="esfera">
-    <inertial>
-      <mass value="0.0000001" />
-      <xacro:insert_block name="elevon_inertia" />
-    </inertial>
-    <visual>
-      <geometry>
-        <sphere radius="0.005" />
-      </geometry>
-    </visual>
-  </link>
-   <gazebo reference="esfera">
-    <material>Gazebo/Green</material>
-  </gazebo>
 <!-- Control de altura -->
 <!-- <joint name="world_fixed" type="prismatic">
   <parent link="world"/>
-  <child link="esfera"/>
+  <child link="${namespace}/base_link"/>
   <axis xyz="0 0 1" />
   <origin xyz="0 0 0" rpy="0 0 0" />
   <limit lower="0" upper="50" effort="20000" velocity="20000"/>
-</joint>
-<joint name="CoG" type="fixed">
-  <child link="${namespace}/base_link"/>
-  <parent link="esfera"/>
-  <origin xyz="0 0 .05" rpy="0 0 0" />
-  <axis xyz="0 0 1" />
 </joint> -->
 <!--  Control de Yaw-->
 <joint name="world_fixed" type="continuous">
   <parent link="world"/>
-  <child link="esfera"/>
+  <child link="${namespace}/base_link"/>
   <axis xyz="0 0 1" />
   <origin xyz="0 0 1" rpy="0 0 0" />
 </joint>
-<joint name="CoG" type="fixed">
-  <child link="${namespace}/base_link"/>
-  <parent link="esfera"/>
-  <origin xyz="0 0 .05" rpy="0 0 0" />
-  <axis xyz="0 0 1" />
-</joint>
 <!-- Control de pitch -->
 <!-- <joint name="world_fixed" type="continuous">
   <parent link="world"/>
-  <child link="esfera"/>
+  <child link="${namespace}/base_link"/>
   <axis xyz="1 0 0" />
   <origin xyz="0 0 1" rpy="0 0 0" />
-</joint>
-<joint name="CoG" type="fixed">
-  <child link="${namespace}/base_link"/>
-  <parent link="esfera"/>
-  <origin xyz="0 0 .05" rpy="0 0 0" />
-  <axis xyz="1 0 0" />
 </joint> -->
 <!-- Contro de Roll -->
-  <!-- <joint name="world_fixed" type="continuous">
-    <parent link="world"/>
-    <child link="esfera"/>
-    <axis xyz="0 1 0" />
-    <origin xyz="0 0 1" rpy="0 0 0" />
-  </joint>
-  <joint name="CoG" type="fixed">
-    <child link="${namespace}/base_link"/>
-    <parent link="esfera"/>
-    <origin xyz="0 0 .05" rpy="0 0 0" />
-    <axis xyz="0 1 0" />
-  </joint> -->
+<!-- <joint name="world_fixed" type="continuous">
+  <parent link="world"/>
+  <child link="${namespace}/base_link"/>
+  <axis xyz="0 1 0" />
+  <origin xyz="0 0 1" rpy="0 0 0" />
+</joint> -->
 </robot>

Commit message: liberado el drone del mundo

File: rotors_description/urdf/kamikaze.xacro (robot description, xacro)
@@ -1,5 +1,5 @@
 <?xml version="1.0"?>
 <robot name="kamikaze" xmlns:xacro="http://ros.org/wiki/xacro">
-  <link name="world"/>
+  <!-- <link name="world"/> -->
   <!-- Included URDF kamikaze properties -->
   <xacro:include filename="$(find rotors_description)/urdf/kamikaze_liftDrag_path.xacro" />
@@ -223,10 +223,10 @@
 </joint> -->
 <!--  Control de Yaw-->
-<joint name="world_fixed" type="continuous">
+<!-- <joint name="world_fixed" type="continuous">
   <parent link="world"/>
   <child link="${namespace}/base_link"/>
   <axis xyz="0 0 1" />
   <origin xyz="0 0 1" rpy="0 0 0" />
-</joint>
+</joint>   -->
 <!-- Control de pitch -->
 <!-- <joint name="world_fixed" type="continuous">
